File: pcb/avionics.kicad_pcb (KiCad board)
At the start: 2 copper layers, 89.5 x 48 mm, 111 parts, among them IC101 STM32F405VGT, IC102 ADP3335, IC201 MAX-7Q, IC701 ADXL345, IC702 L3G4200D, IC703 MS5611-01BA03, IC704 HMC5883L, M3_MOUNT VAL**, P101 CONN_01X02, P102 CONN_01X04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

Commit message: WE'RE FINALLY DONE!!!
Routing:
- net GND: track 225.1 -> 329.5 mm, vias 33 -> 82
Changed lines of the file:
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@@
     (links 290)
     (no_connects 0)
-    (area 87.949999 40.949999 188.050001 89.050001)
+    (area 94.982429 39.925 191.268334 89.925)
     (thickness 1.6)
     (drawings 4)
-    (tracks 1346)
+    (tracks 1450)
     (zones 0)
     (modules 111)
@@
   (segment (start 156.9212 60.3642) (end 156.4778 60.3642) (width 0.5) (layer F.Cu) (net 2))
   (segment (start 156.9212 60.3642) (end 156.501 60.3642) (width 0.5) (layer F.Cu) (net 2))
+  (segment (start 121 43) (end 119 43) (width 0.5) (layer F.Cu) (net 3))
+  (via (at 107 43) (size 0.8) (layers F.Cu B.Cu) (net 3))
+  (segment (start 107 43) (end 109 43) (width 0.5) (layer F.Cu) (net 3))
+  (via (at 109 43) (size 0.8) (layers F.Cu B.Cu) (net 3))
+  (segment (start 109 43) (end 111 43) (width 0.5) (layer B.Cu) (net 3))
+  (via (at 111 43) (size 0.8) (layers F.Cu B.Cu) (net 3))
+  (segment (start 111 43) (end 113 43) (width 0.5) (layer F.Cu) (net 3))
+  (via (at 113 43) (size 0.8) (layers F.Cu B.Cu) (net 3))
+  (segment (start 113 43) (end 115 43) (width 0.5) (layer B.Cu) (net 3))
+  (via (at 115 43) (size 0.8) (layers F.Cu B.Cu) (net 3))
+  (segment (start 115 43) (end 117 43) (width 0.5) (layer F.Cu) (net 3))
+  (via (at 117 43) (size 0.8) (layers F.Cu B.Cu) (net 3))
+  (segment (start 117 43) (end 119 43) (width 0.5) (layer B.Cu) (net 3))
+  (via (at 119 43) (size 0.8) (layers F.Cu B.Cu) (net 3))
+  (via (at 107 45) (size 0.8) (layers F.Cu B.Cu) (net 3))
+  (segment (start 107 43) (end 107 45) (width 0.5) (layer B.Cu) (net 3))
+  (via (at 121 43) (size 0.8) (layers F.Cu B.Cu) (net 3))
+  (via (at 110 51) (size 0.8) (layers F.Cu B.Cu) (net 3))
+  (via (at 110 53) (size 0.8) (layers F.Cu B.Cu) (net 3))
+  (segment (start 110 53) (end 109 54) (width 0.5) (layer B.Cu) (net 3))
+  (segment (start 109 54) (end 109 55) (width 0.5) (layer B.Cu) (net 3))
+  (segment (start 109 57) (end 109 55) (width 0.5) (layer F.Cu) (net 3))
+  (via (at 109 55) (size 0.8) (layers F.Cu B.Cu) (net 3))
+  (segment (start 110 53) (end 110 51) (width 0.5) (layer F.Cu) (net 3))
+  (segment (start 119 57) (end 121 57) (width 0.5) (layer B.Cu) (net 3))
+  (via (at 121 59) (size 0.8) (layers F.Cu B.Cu) (net 3))
+  (segment (start 121 57) (end 121 59) (width 0.5) (layer F.Cu) (net 3))
+  (via (at 121 57) (size 0.8) (layers F.Cu B.Cu) (net 3))
+  (segment (start 119 55) (end 119 57) (width 0.5) (layer F.Cu) (net 3))
+  (via (at 119 57) (size 0.8) (layers F.Cu B.Cu) (net 3))
+  (via (at 105 59) (size 0.8) (layers F.Cu B.Cu) (net 3))
+  (segment (start 107 59) (end 105 59) (width 0.5) (layer F.Cu) (net 3))
+  (via (at 107 59) (size 0.8) (layers F.Cu B.Cu) (net 3))
+  (segment (start 109 59) (end 107 59) (width 0.5) (layer B.Cu) (net 3))
+  (via (at 109 59) (size 0.8) (layers F.Cu B.Cu) (net 3))
+  (segment (start 111 59) (end 109 59) (width 0.5) (layer F.Cu) (net 3))
+  (via (at 111 59) (size 0.8) (layers F.Cu B.Cu) (net 3))
+  (segment (start 113 59) (end 111 59) (width 0.5) (layer B.Cu) (net 3))
+  (via (at 113 59) (size 0.8) (layers F.Cu B.Cu) (net 3))
+  (segment (start 115 59) (end 113 59) (width 0.5) (layer F.Cu) (net 3))
+  (via (at 115 59) (size 0.8) (layers F.Cu B.Cu) (net 3))
+  (segment (start 117 59) (end 115 59) (width 0.5) (layer B.Cu) (net 3))
+  (via (at 117 59) (size 0.8) (layers F.Cu B.Cu) (net 3))
+  (segment (start 119 59) (end 117 59) (width 0.5) (layer F.Cu) (net 3))
+  (via (at 119 59) (size 0.8) (layers F.Cu B.Cu) (net 3))
+  (segment (start 119 57) (end 119 59) (width 0.5) (layer B.Cu) (net 3))
+  (segment (start 119 51) (end 119 49) (width 0.5) (layer B.Cu) (net 3))
+  (via (at 119 51) (size 0.8) (layers F.Cu B.Cu) (net 3))
+  (segment (start 119 53) (end 119 51) (width 0.5) (layer F.Cu) (net 3))
+  (via (at 119 53) (size 0.8) (layers F.Cu B.Cu) (net 3))
+  (segment (start 119 55) (end 119 53) (width 0.5) (layer B.Cu) (net 3))
+  (via (at 119 55) (size 0.8) (layers F.Cu B.Cu) (net 3))
+  (segment (start 119 49) (end 117 49) (width 0.5) (layer B.Cu) (net 3))
+  (segment (start 117 49) (end 119 49) (width 0.5) (layer B.Cu) (net 3))
+  (via (at 119 49) (size 0.8) (layers F.Cu B.Cu) (net 3))
+  (segment (start 119 49) (end 117 49) (width 0.5) (layer F.Cu) (net 3))
+  (segment (start 115 57) (end 117 57) (width 0.5) (layer F.Cu) (net 3))
+  (segment (start 117 49) (end 117 47) (width 0.5) (layer B.Cu) (net 3))
+  (via (at 117 49) (size 0.8) (layers F.Cu B.Cu) (net 3))
+  (segment (start 117 51) (end 117 49) (width 0.5) (layer F.Cu) (net 3))
+  (via (at 117 51) (size 0.8) (layers F.Cu B.Cu) (net 3))
+  (segment (start 117 53) (end 117 51) (width 0.5) (layer B.Cu) (net 3))
+  (via (at 117 53) (size 0.8) (layers F.Cu B.Cu) (net 3))
+  (segment (start 117 55) (end 117 53) (width 0.5) (layer F.Cu) (net 3))
+  (via (at 117 55) (size 0.8) (layers F.Cu B.Cu) (net 3))
+  (segment (start 117 57) (end 117 55) (width 0.5) (layer B.Cu) (net 3))
+  (via (at 117 57) (size 0.8) (layers F.Cu B.Cu) (net 3))
+  (segment (start 115 47) (end 115 49) (width 0.5) (layer F.Cu) (net 3))
+  (via (at 105 57) (size 0.8) (layers F.Cu B.Cu) (net 3))
+  (segment (start 107 57) (end 105 57) (width 0.5) (layer B.Cu) (net 3))
+  (via (at 107 57) (size 0.8) (layers F.Cu B.Cu) (net 3))
+  (segment (start 109 57) (end 107 57) (width 0.5) (layer F.Cu) (net 3))
+  (via (at 109 57) (size 0.8) (layers F.Cu B.Cu) (net 3))
+  (segment (start 111 57) (end 109 57) (width 0.5) (layer B.Cu) (net 3))
+  (via (at 111 57) (size 0.8) (layers F.Cu B.Cu) (net 3))
+  (segment (start 113 57) (end 111 57) (width 0.5) (layer F.Cu) (net 3))
+  (via (at 113 57) (size 0.8) (layers F.Cu B.Cu) (net 3))
+  (segment (start 115 57) (end 113 57) (width 0.5) (layer B.Cu) (net 3))
+  (via (at 115 57) (size 0.8) (layers F.Cu B.Cu) (net 3))
+  (segment (start 115 55) (end 115 57) (width 0.5) (layer F.Cu) (net 3))
+  (via (at 115 55) (size 0.8) (layers F.Cu B.Cu) (net 3))
+  (segment (start 115 53) (end 115 55) (width 0.5) (layer B.Cu) (net 3))
+  (via (at 115 53) (size 0.8) (layers F.Cu B.Cu) (net 3))
+  (segment (start 115 51) (end 115 53) (width 0.5) (layer F.Cu) (net 3))
+  (via (at 115 51) (size 0.8) (layers F.Cu B.Cu) (net 3))
+  (segment (start 115 49) (end 115 51) (width 0.5) (layer B.Cu) (net 3))
+  (via (at 115 49) (size 0.8) (layers F.Cu B.Cu) (net 3))
+  (segment (start 107 45) (end 109 45) (width 0.5) (layer B.Cu) (net 3))
+  (segment (start 106.25 45.75) (end 107 45) (width 0.5) (layer B.Cu) (net 3))
+  (segment (start 106.25 46.55) (end 106.25 45.75) (width 0.5) (layer B.Cu) (net 3))
+  (segment (start 113 45) (end 115 45) (width 0.5) (layer F.Cu) (net 3))
+  (via (at 113 45) (size 0.8) (layers F.Cu B.Cu) (net 3))
+  (segment (start 111 45) (end 113 45) (width 0.5) (layer B.Cu) (net 3))
+  (via (at 111 45) (size 0.8) (layers F.Cu B.Cu) (net 3))
+  (segment (start 109 45) (end 111 45) (width 0.5) (layer F.Cu) (net 3))
+  (via (at 109 45) (size 0.8) (layers F.Cu B.Cu) (net 3))
+  (via (at 115 45) (size 0.8) (layers F.Cu B.Cu) (net 3))
+  (via (at 117 47) (size 0.8) (layers F.Cu B.Cu) (net 3))
+  (segment (start 117 45) (end 117 47) (width 0.5) (layer F.Cu) (net 3))
+  (via (at 117 45) (size 0.8) (layers F.Cu B.Cu) (net 3))
+  (segment (start 115 45) (end 117 45) (width 0.5) (layer B.Cu) (net 3))
+  (segment (start 117 47) (end 115 47) (width 0.5) (layer B.Cu) (net 3))
+  (via (at 115 47) (size 0.8) (layers F.Cu B.Cu) (net 3))
+  (segment (start 115 47) (end 115 45) (width 0.5) (layer F.Cu) (net 3))
+  (via (at 106.25 46.55) (size 0.8) (layers F.Cu B.Cu) (net 3))
+  (segment (start 106.25 46.55) (end 106.3 46.6) (width 0.5) (layer B.Cu) (net 3))
   (segment (start 105 48.2) (end 106 47.2) (width 0.5) (layer F.Cu) (net 3))
   (via (at 105 48.2) (size 0.8) (layers F.Cu B.Cu) (net 3))
   (segment (start 103.0815 50.1185) (end 105 48.2) (width 1) (layer F.Cu) (net 3))
-  (via (at 107.2 45) (size 0.8) (layers F.Cu B.Cu) (net 3))
-  (segment (start 107.2 45.6) (end 107.2 45) (width 0.5) (layer F.Cu) (net 3))
-  (segment (start 106 46.8) (end 107.2 45.6) (width 0.5) (layer F.Cu) (net 3))
+  (segment (start 106 46.8) (end 106.25 46.55) (width 0.5) (layer F.Cu) (net 3))
   (segment (start 106 47.2) (end 106 46.8) (width 0.5) (layer F.Cu) (net 3))
   (segment (start 101.2 76.0815) (end 101.2 77.6) (width 1) (layer F.Cu) (net 3))
